Commit message: URDF fixup

File: SpotSim/URDF/spot-front-left.urdf (robot description, URDF)
Before this commit: robot C:/Users/Michael Student/Downloads/spot.urdf, 4 links, 4 joints
Joints:
- joint front left shoulder abduction motor: origin xyz=0.1935 -1.326719 0.628594 rpy=1.5708 -0.00001 -1.570793 -> xyz=0.365 0.0528 0.012301 rpy=1.5708 -0.00001 -1.570793

File: SpotSim/URDF/spot-front-right.urdf (robot description, URDF)
Before this commit: robot C:/Users/Michael Student/Downloads/spot.urdf, 4 links, 4 joints
Joints:
- joint front right shoulder abduction motor: origin xyz=0.5335 -1.432319 0.628595 rpy=1.5708 -0.00001 -1.570793 -> xyz=0.365 -0.0528 0.012301 rpy=1.5708 -0.00001 -1.570793

File: SpotSim/URDF/spot-rear-left.urdf (robot description, URDF)
Before this commit: robot C:/Users/Michael Student/Downloads/spot.urdf, 5 links, 4 joints
Joints:
- joint rear left shoulder abduction motor: origin xyz=-0.4784 -1.326719 0.628494 rpy=1.5708 -0.00001 -1.570793 -> xyz=-0.3084 0.0528 0.012301 rpy=1.5708 -0.00001 -1.570793

File: SpotSim/URDF/spot-rear-right.urdf (robot description, URDF)
Before this commit: robot C:/Users/Michael Student/Downloads/spot.urdf, 34 links, 33 joints
Links:
- removed link accelerometer
- removed link front left forearm
- removed link front left shoulder
- removed link front left upperarm
- removed link front right forearm
- removed link front right shoulder
- removed link front right upperarm
- removed link gps
- removed link gyro
- removed link inertial unit
- removed link left bottom led
- removed link left flank camera
- removed link left head camera
- removed link left middle down led
- removed link left middle up led
- removed link left top led
- removed link rear camera
- removed link rear left forearm
- removed link rear left shoulder
- removed link rear left upperarm
- removed link right bottom led
- removed link right flank camera
- removed link right head camera
- removed link right middle down led
- removed link right middle up led
- removed link right top led
- removed link solid_0
- removed link solid_1
- removed link solid_2
Joints:
- removed joint base_link_accelerometer_joint
- removed joint base_link_gps_joint
- removed joint base_link_gyro_joint
- removed joint base_link_inertial unit_joint
- removed joint base_link_left bottom led_joint
- removed joint base_link_left flank camera_joint
- removed joint base_link_left head camera_joint
- removed joint base_link_left middle down led_joint
- removed joint base_link_left middle up led_joint
- removed joint base_link_left top led_joint
- removed joint base_link_rear camera_joint
- removed joint base_link_right bottom led_joint
- removed joint base_link_right flank camera_joint
- removed joint base_link_right head camera_joint
- removed joint base_link_right middle down led_joint
- removed joint base_link_right middle up led_joint
- removed joint base_link_right top led_joint
- removed joint front left elbow motor
- removed joint front left piston motor
- removed joint front left shoulder abduction motor
- removed joint front left shoulder rotation motor
- removed joint front right elbow motor
- removed joint front right piston motor
- removed joint front right shoulder abduction motor
- removed joint front right shoulder rotation motor
- removed joint rear left elbow motor
- removed joint rear left piston motor
- removed joint rear left shoulder abduction motor
- removed joint rear left shoulder rotation motor

Commit message: Spot sims first steps

File: SpotSim/URDF/spot-front-left.urdf (robot description, URDF)
Before this commit: robot C:/Users/Michael Student/Downloads/spot.urdf, 4 links, 4 joints
Joints:
- removed joint front left piston motor
